File: hardware/PKG900000001531.sch (EAGLE design)
At the start: 293 parts, among them IC1 CAT24C256YI-G, IC2 FT232RQ, IC3 TPS62111, IC5 FT232RQ, IC6 SN74LVC1G126DCKR, IC7 SN74LVC1G126DCKR, J1 JST-GH-5H, J10 FPC-15VERT, J11 FPC-15VERT, J12 JST-GH-6H, J13 JST-GH-6H, J14 JST-GH-4H, J2 DF40HC(3.0)-100DS-0.4V(51), J3 USD_WURTH, J4 DIP-1, J5 SM10B-SRSS-TB, J7 USB-TYPE-C, J8 DF40HC(3.0)-100DS-0.4V(51), J9 CON8X3STD, Q1 FDN360P, Q2 DNP, Q3 FDN360P, Q4 FDN360P, Q6 FDN360P, U1 TPS2041BDGN, U10 DNP, U100 STM32H753II, U101 MIC94081, U102 USB2513, U105 TPS2121, U106 FM25V02A-DG, U107 TPD4E02B0410-USON, U108 BMP388, U109 MIC94081, U11 ICM-20602, U110 TCR2EF18, U13 USB3300-EZK-TR, U15 BMI088, U16 MIC94081, U17 TPD4E02B0410-USON, U18 TPD4E02B0410-USON, U2 TJA1051TK/3, U25 TPS2041BDGN, U26 TS3USB30, U3 TPD4E02B0410-USON, U4 EVQ, U5 G313-06329-00, U6 NCP308, U7 ICM-42605, U8 TPD4E02B0410-USON, U9 BMM150, Y1 24.000MHz, Y2 16.000MHz, Y3 32.768KHz CL6, Y4 24.000MHz

Commit message: Update hardware files for revision 2.
Parts:
- added R13, R47, R55, R56: 10K 1%, qualified_1:R0201
- added R46: DNP, qualified_1:R0201
- added R52, R54: 0R, qualified_1:R0201
- added U30: TS3A5223, qualified_1:TS3A5223
- R77: value DNP -> 10K 1%
- U$2: BOARD PCB900000001531v1 -> PCB900000001531v2; TITLE CM4 + Pixhawk FMUv6 -> RPi CM4 + Pixhawk FMUv6
- renumbered U4 to S3
Connections:
- removed net 3V3_SPEKTRUM$1: U16.VOUT
- removed net 5.USB_DEVICE_VBUS: FB4.1
- removed net 6.USB_DEVICE_VBUS: FB1.1
- new net 3V3_SPEKTRUM: J1.P$4, U16.VOUT
- new net BMM150_PS: R46.2, R47.1, U9.PS@A1
- new net UART_MUX_SEL$: R55.1, R56.2, U30.SEL1, U30.SEL2
- new net USART3_RX_DEBUG_FTDI: IC6A.O, U30.NO1
- new net USART3_RX_DEBUG_JST: D5.A, U30.NC1
- new net USART3_TX_DEBUG_FTDI: IC5.RXD, U30.NO2
- new net USART3_TX_DEBUG_JST: J5.2, U3.P1, U30.NC2
- net 2.3.3V_VCC_3.3: now also U30.VCC; no longer J1.P$4
- net 3V3_SENSORS: now also R47.2
- net 7.UART4_4W_RXD: now also R54.1
- net 7.UART4_4W_TXD: now also R52.1
- net BTN_A$22: now also S1.B
- net GND: now also R13.1, R46.1, R56.1, S1.A', U30.GND; no longer U9.PS@A1
- net SDO$1: now also R13.2
- net UART5_CTS_TELEM2: now also R1.2, R2.2
- net UART5_RTS_TELEM2: now also R3.2, R4.2
- net UART5_RX_TELEM2: now also R52.2
- net UART5_TX_TELEM2: now also R54.2
- net UART7_CTS_TELEM1: no longer R1.2, R2.2
- net UART7_RTS_TELEM1: no longer R3.2, R4.2
- net USART3_RX_DEBUG: now also U30.COM1; no longer D5.A, IC6A.O
- net USART3_TX_DEBUG: now also U30.COM2; no longer IC5.RXD, J5.2, U3.P1
- net VBUS_SENSE: now also FB1.1, FB4.1, R55.2
Other:
- note added: "1"
- note added: "2"
- note added: "2020-10-17"
- note added: "2020-11-30"
- note added: "23) JST GH 6-pin (GPS) Header"
- note added: "24) JST GH 6-pin (Power) Header"
- note added: "26) JST GH 4-pin (CAN) Header"
- note added: "27) JST GH 5-pin (RC) Header"
- note added: "ACS"
- note added: "Fixed USB-UART power supply and debug mux. Populated the BMP388 chip. Set up BMM150 for I2C. Added orientation arrow."
- note added: "Initial design - https://geppetto.gumstix.com/#\!/design/8869/"
- note added: "JST GH 4-pin (CAN) Header"
- note added: "JST GH 5-pin (RC) Header"
- note added: "JST GH 6-pin (GPS) Header"
- note added: "JST GH 6-pin (Power) Header"
- note added: "RPi CM4 + Pixhawk FMUv6"
- note removed: "23) JST GH 6-pin Vertical Header"
- note removed: "24) JST GH 6-pin Vertical Header"
- note removed: "26) JST GH Vertical 4-pin Header"
- note removed: "27) Custom 5-pin Header (JST-GH)"
- note removed: "CM4 + Pixhawk FMUv6"
- note removed: "Custom 5-pin Header (JST-GH)"
- note removed: "JST GH 6-pin Vertical Header"
- note removed: "JST GH Vertical 4-pin Header"

Commit message: Update board design files to v4.
Add ROS2 and Coral support information to the firmware docs.
Parts:
- removed C103: 0.1uF, qualified_1@eagle_src_repo_a6c39d613d14f2251c563284af21e76ddd4db3e9:C0201
- removed C242, C272, C273: 0.1uF, qualified_1:C0201
- removed C264: 1.0uF, qualified_1:C0402
- removed J4: DIP-1, qualified_1:DIP-1
- removed Q2: DNP, qualified_1:BSS138
- removed R116: DNP, qualified_1:R0201
- removed R118, R121, R122: 0R, qualified_1:R0201
- removed U102: USB2513, qualified_1:USB2513
- removed U110: TCR2EF18, qualified_1:TCR2EF18
- removed U26: TS3USB30, qualified_1:TS3USB30WQ
- added C158, C167: 10uF, qualified_1:C0603
- added C31, C96: 1.0uF, qualified_1:C0402
- added C32: 10pF, qualified_1:C0201
- added C72, C73, C74, C75, C76, C77, C78, C79, C82, C83, C84, C85, C86, C88, C89, C92, C93, C95, C97: 0.1uF, qualified_1:C0201
- added C90, C91: 4.7uF / 16V, qualified_1:C0603
- added C94: 6.8nF, qualified_1:C0201
- added R58: 0R, qualified_1:R0201
- added R68: 5K1, qualified_1:R0201
- added R69, R70: 10K 1%, qualified_1:R0201
- added U12: ADP1740ACPZ-1.2-R7, qualified_1:ADP174X
- added U14: USB2517-JZX, qualified_1:USB2517-JZX
- added U19: (no value), qualified_1:TXS0104E
- added U4: ASM1142, qualified_1:ASM1142
- added Y5: 20.000MHz, qualified_1:Y4CRYSTAL-3225
- C13: value 1.0uF -> 0.1uF; device qualified_1:C0402 -> qualified_1:C0201; DM (none) -> 0; DR (none) -> 90.000; DX (none) -> 5.600; DY (none) -> 28.400; SHEETNO (none) -> 2
- C16: value 1.0uF -> 0.1uF; device qualified_1:C0402 -> qualified_1:C0201
- C2: value DNP -> 4.7nF; device qualified_1:C0402 -> qualified_1:C0201
- R11: value 10K 1% -> 12K1
- R117: value DNP -> 10K 1%
- R20: value DNP -> 1K5
- R27, R28: value 10K 1% -> 1K5; device qualified_1@eagle_src_repo_a6c39d613d14f2251c563284af21e76ddd4db3e9:R0201 -> qualified_1:R0201
- R43, R9: value DNP -> 0R
- R5: value 0R -> 100K 1%; DM (none) -> 0; DR (none) -> -270.000; DX (none) -> -20.800; DY (none) -> 8.200; SHEETNO (none) -> 9
- RT4, RT5: value DNP -> 60R4
- U$2: device qualified_1:GEPPETTO_LABEL_SMALL -> qualified_1:UPVERTER_LABELSMALL; BOARD PCB900000001531v2 -> PCB900000001531v4; TITLE RPi CM4 + Pixhawk FMUv6 -> RPi CM4 + Pixhawk FMUv6U; YEAR 2020 -> 2021
- U6: value NCP308 -> (none)
Connections:
- removed net !PCIE_CLKREQ$17: Q2.S, R116.2, R20.2, U5.!CLKREQ
- removed net 1.USB_HS_VBUS: U13.VBUS
- removed net 1.USB_MUX_D_N: U102.USBDM_DN1, U26.D-
- removed net 1.USB_MUX_D_P: U102.USBDP_DN1, U26.D+
- removed net 7.PCIE_CLK_N: R121.2, U5.PCIE_REFCLK_N
- removed net 7.PCIE_CLK_P: R118.2, U5.PCIE_REFCLK_P
- removed net CC$3: J7.CC1, J7.CC2, R89.2
- removed net INTR$17: U5.INTR
- removed net PCIE_TX_N$17: U5.PCIE_TX_N
- removed net PCIE_TX_P$17: U5.PCIE_TX_P
- removed net RPIBOOT_SWITCH$7: R11.2, S2.A, S2.A'
- removed net SELECT: J4.2, R27.2, U26.S
- removed net USBMUX_OE$13: R28.2, U26.!OE
- removed net USB_CRFILT$4: C13.1, C272.1, U102.CRFILT
- removed net USB_PLLFILT$4: C242.1, C264.1, U102.PLLFILT
- removed net USB_VBUS_DET$4: R97.2, U102.VBUS_DET
- removed net V1.8$17: C16.1, Q2.G, R116.1, R19.2, R21.2, R43.2, R48.2, U110.VOUT
- new net !INT: U4.!SMI
- new net !PCIE_WAKE: U4.!PEWAKE
- new net !RST$: R70.1, U4.!PORST
- new net !SPI_CS$: U4.!SPI_CS
- new net !USB1_NOC: U4.!OC1
- new net !USB2_NOC: U4.!OC2
- new net 7.GPIO2_GPIO: J8.58, U19.B3
- new net 7.GPIO3_GPIO: J8.56, U19.B4
- new net 7.GPIO6_GPIO: J8.30, U19.B2
- new net 7.GPIO7_GPIO: J8.37, U19.B1
- new net 7.PCIE_NRESET: J2.9, R69.1, U4.!PERST
- new net CC1$3: J7.CC1, R68.2
- new net CC2$3: J7.CC2, R89.2
- new net CFG_SEL2$: R5.2, U14.CFG_SEL2
- new net I2C_SCL: R27.1, U19.A4, U5.RESERVED@50
- new net I2C_SDA: R28.1, U19.A3, U5.RESERVED@49
- new net PCIE_CLK_N: J2.12, U4.PCIE_REFCLK_N
- new net PCIE_CLK_P: J2.10, U4.PCIE_REFCLK_P
- new net PCIE_RX0__N: C93.2, U4.PCIE_TX0_N
- new net PCIE_RX0__P: C92.2, U4.PCIE_TX0_P
- new net PCIE_TX_N: J2.24, U4.PCIE_RX0_P
- new net PCIE_TX_P: J2.22, U4.PCIE_RX0_N
- new net PHY_PRG: U19.A1, U5.RESERVED@84
- new net REXT$: R11.2, U4.REXT
- new net RPIBOOT_SWITCH$19: R20.2, S2.A, S2.A'
- new net SPI_CLK$: U4.SPI_CLK
- new net SPI_DI$: U4.SPI_DI
- new net SPI_DO$: U4.SPI_DO
- new net UART_RX$: U4.UART_RX
- new net UART_TX$: U4.UART_TX
- new net USB1_N: U4.USB1_N, U5.USB2_D_N
- new net USB1_P: U4.USB1_P, U5.USB2_D_P
- new net USB1_PWREN: U4.PWRON1
- new net USB1_SSRX_N: U4.USB1_SSRX_N, U5.PCIE_TX_N
- new net USB1_SSRX_P: U4.USB1_SSRX_P, U5.PCIE_TX_P
- new net USB1_SSTX_N: C16.2, U4.USB1_SSTX_N
- new net USB1_SSTX_P: C72.2, U4.USB1_SSTX_P
- new net USB1_SSTX__N: C16.1, U5.PCIE_RX_P
- new net USB1_SSTX__P: C72.1, U5.PCIE_RX_N
- new net USB2_N: U4.USB2_N
- new net USB2_P: U4.USB2_P
- new net USB2_PWREN: U4.PWRON2
- new net USB2_SSRX_N: U4.USB2_SSRX_N
- new net USB2_SSRX_P: U4.USB2_SSRX_P
- new net USB2_SSTX_N: U4.USB2_SSTX_N
- new net USB2_SSTX_P: U4.USB2_SSTX_P
- new net USB_CRFILT$: C31.1, C95.1, U14.VDD18
- new net USB_PLLFILT$: C96.1, C97.1, U14.VDD18PLL
- new net V1.2$: C167.1, C74.1, C75.1, C78.1, C79.1, C82.1, C83.1, C84.1, C89.1, C90.1, C91.1, U12.SENSE, U12.VOUT, U4.VDD, U4.VDDP, U4.VDDSUS, U4.VDDU
- new net VBUS_DET$: R97.2, U14.VBUS_DET
- new net VCC1V1_SS$: C94.1, U12.SS
- new net XI$: C32.2, U4.XI, Y5.1
- new net XO$: C32.1, U4.XO, Y5.3
- new net _PCIE_CLK_N: R43.2, U5.PCIE_REFCLK_N
- new net _PCIE_CLK_P: R58.2, U5.PCIE_REFCLK_P
- net 1.USB_HS_D_N: now also U14.USBDN1_DM/PRT_DIS_M1; no longer U26.D2-
- net 1.USB_HS_D_P: now also U14.USBDN1_DP/PRT_DIS_P1; no longer U26.D2+
- net 2.3.3V_VCC_3.3: now also C13.1, C158.1, C73.1, C76.1, C77.1, C85.1, C86.1, C88.1, R5.1, R69.2, R70.2, R91.1, U12.EN, U12.VIN, U14.VDD33, U14.VDD33CR, U14.VDD33PLL, U14.VDDA33, U14.VDDA33_2, U14.VDDA33_3, U14.VDDA33_4, U4.VCC, U4.VCCP, U4.VCCSUS, U4.VCCU; no longer C103.1, J4.1, U102.VDD33@10, U102.VDD33@15, U102.VDD33@23, U102.VDD33@29, U102.VDD33@36, U102.VDD33@5, U26.VCC
- net 4.USB_D_N: now also U14.USBUP_DM; no longer U102.USBDM_UP
- net 4.USB_D_P: now also U14.USBUP_DP; no longer U102.USBDP_UP
- net 5.USB_DEVICE_D_N: now also U14.USBDN6_DM/PRT_DIS_M6; no longer U102.USBDM_DN2
- net 5.USB_DEVICE_D_P: now also U14.USBDN6_DP/PRT_DIS_P6; no longer U102.USBDP_DN2
- net 6.USB_DEVICE_D_N: now also U14.USBDN7_DM/PRT_DIS_M7; no longer U102.USBDM_DN3
- net 6.USB_DEVICE_D_P: now also U14.USBDN7_DP/PRT_DIS_P7; no longer U102.USBDP_DN3
- net 7.1.8V_VCC_1.8: now also C34.1, R19.2, R21.2, R27.2, R28.2, R48.2, U19.OE, U19.VCCA, U5.AON; no longer R43.1
- net 7.3.3V_VCC_3.3: now also U19.VCCB; no longer C273.1, C34.1, R9.1, U110.CONTROL, U110.VIN, U5.AON
- net 7.PCIE_CLKREQ_GPIO: now also R9.1; no longer Q2.D, R9.2
- net CORAL_D_N: now also J2.3, U14.USBDN5_DM/PRT_DIS_M5; no longer J2.5, U5.USB2_D_N
- net CORAL_D_P: now also J2.5, U14.USBDN5_DP/PRT_DIS_P5; no longer J2.3, U5.USB2_D_P
- net GND: now also C158.2, C167.2, C31.2, C73.2, C74.2, C75.2, C76.2, C77.2, C78.2, C79.2, C82.2, C83.2, C84.2, C85.2, C86.2, C88.2, C89.2, C90.2, C91.2, C94.2, C95.2, C96.2, C97.2, R43.1, R58.1, R68.1, R9.2, U12.GND, U14.EPAD, U14.TEST, U19.GND, U4.GND, Y5.2, Y5.4; no longer C103.2, C16.2, C242.2, C264.2, C272.2, C273.2, R118.1, R121.1, R122.1, R27.1, R28.1, R5.1, R91.1, U102.VSS, U110.GND, U26.GND
- net PCIE_RX_N: now also C92.1, J2.18; no longer R5.2, U5.PCIE_RX_N
- net PCIE_RX_P: now also C93.1, J2.16; no longer R122.2, U5.PCIE_RX_P
- net PMIC_EN$17: now also U19.A2
- net USB_D_N: now also U14.USBDN2_DM/PRT_DIS_M2; no longer U26.D1-
- net USB_D_P: now also U14.USBDN2_DP/PRT_DIS_P2; no longer U26.D1+
- net USB_HS_IND$4: now also U14.HS_IND/CFG_SEL1; no longer U102.HS_IND/CFG_SEL1
- net USB_NRESET$4: now also U14.RESET_N; no longer U102.RESET_N
- net USB_RBIAS$4: now also U14.RBIAS; no longer U102.RBIAS
- net USB_SCL$4: now also U14.SCL/SMBCLK/CFG_SEL0; no longer U102.SCL/CFG_SEL0
- net USB_SDA$4: now also U14.SDA/SMBDATA/NON_REM1; no longer U102.SDA/NON_REM1
- net USB_SUSP_IND$4: now also U14.SUSP_IND/LOCAL_PWR/NON_REM0; no longer U102.SUSP_IND/NON_REM0
- net USB_XTAL1$4: now also U14.XTAL1/CLKIN; no longer U102.XTALIN
- net USB_XTAL2$4: now also U14.XTAL2; no longer U102.XTALOUT
- net VBUS_SENSE: now also U13.VBUS
Other:
- note added: "14) 7-Port USB Client Hub"
- note added: "2021-01-12"
- note added: "2021-04-01"
- note added: "3"
- note added: "32) PCIe to USB3.0"
- note added: "4"
- note added: "7-Port USB Client Hub"
- note added: "Add PCIe->USB3 and interface to Coral. Change to 7-port hub to allow flashing of CM4."
- note added: "Fix USB polarity to Coral and add PCIe connections."
- note added: "PCIe to USB3.0"
- note removed: "14) 3-Port USB Client Hub"
- note removed: "3-Port USB Client Hub"
- note removed: "32) USB 2-Port Switch"
- note removed: "USB 2-Port Switch"
